File: luis48.kicad_sch (KiCad schematic)
At the start: 2 parts, among them M1 Module-ign8-0.2, U1 ISL9V3040D3ST-F085C

Commit message: correjido
Parts:
- added U2: 5007620481, jlc_footprints:CONN-TH_5007620481, symbol jlc_parts:5007620481
Changed lines of the file:
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@@
 	(paper "A4")
+	(symbol
+		(lib_id "jlc_parts:5007620481")
+		(at 214.63 76.2 0)
+		(unit 1)
+		(exclude_from_sim no)
+		(in_bom yes)
+		(on_board yes)
+		(dnp no)
+		(fields_autoplaced yes)
+		(property "Reference" "U2"
+			(at 214.63 39.37 0)
+			(effects
+				(font
+					(size 1.27 1.27)
+				)
+			)
+		)
+		(property "Value" "5007620481"
+			(at 214.63 41.91 0)
+			(effects
+				(font
+					(size 1.27 1.27)
+				)
+			)
+		)
+		(property "Footprint" "jlc_footprints:CONN-TH_5007620481"
+			(at 214.63 86.36 0)
+			(effects
+				(font
+					(size 1.27 1.27)
+					(italic yes)
+				)
+				(hide yes)
+			)
+		)
+		(property "Datasheet" "https://atta.szlcsc.com/upload/public/pdf/source/20180207/C164171_15179949969151359204.pdf"
+			(at 212.344 76.073 0)
+			(effects
+				(font
+					(size 1.27 1.27)
+				)
+				(justify left)
+				(hide yes)
+			)
+		)
+		(property "Description" ""
+			(at 214.63 76.2 0)
+			(effects
+				(font
+					(size 1.27 1.27)
+				)
+				(hide yes)
+			)
+		)
+		(property "LCSC" "C164171"
+			(at 214.63 76.2 0)
+			(effects
+				(font
+					(size 1.27 1.27)
+				)
+				(hide yes)
+			)
+		)
+		(pin "13"
+		)
+		(pin "10"
+		)
+		(pin "12"
+		)
+		(pin "1"
+		)
+		(pin "11"
+		)
+		(pin "14"
+		)
+		(pin "16"
+		)
+		(pin "17"
+		)
+		(pin "18"
+		)
+		(pin "2"
+		)
+		(pin "15"
+		)
+		(pin "19"
+		)
+		(pin "20"
+		)
+		(pin "21"
+		)
+		(pin "22"
+		)
+		(pin "23"
+		)
+		(pin "24"
+		)
+		(pin "25"
+		)
+		(pin "27"
+		)
+		(pin "28"
+		)
+		(pin "26"
+		)
+		(pin "45"
+		)
+		(pin "44"
+		)
+		(pin "46"
+		)
+		(pin "47"
+		)
+		(pin "5"
+		)
+		(pin "29"
+		)
+		(pin "4"
+		)
+		(pin "40"
+		)
+		(pin "7"
+		)
+		(pin "36"
+		)
+		(pin "39"
+		)
+		(pin "33"
+		)
+		(pin "30"
+		)
+		(pin "35"
+		)
+		(pin "38"
+		)
+		(pin "6"
+		)
+		(pin "41"
+		)
+		(pin "48"
+		)
+		(pin "3"
+		)
+		(pin "34"
+		)
+		(pin "32"
+		)
+		(pin "37"
+		)
+		(pin "42"
+		)
+		(pin "43"
+		)
+		(pin "9"
+		)
+		(pin "8"
+		)
+		(pin "31"
+		)
+		(instances
+			(project "luis48"
+				(path "/fbc7a05b-dc90-4428-b3bf-681204682704"
+					(reference "U2")
+					(unit 1)
+				)
+			)
+		)
+	)
 	(symbol
 		(lib_id "jlc_parts:ISL9V3040D3ST-F085C")

Commit message: wew
Parts:
- removed M1: Module-ign8-0.2, hellen-one-ign8-0.2:ign8, symbol ign8:Module-ign8-0.2
- removed U1: ISL9V3040D3ST-F085C, jlc_footprints:JLC_DPAK_L6.5-W6.0-P2.29-LS9.9-TL, symbol jlc_parts:ISL9V3040D3ST-F085C
- removed U2: 5007620481, jlc_footprints:CONN-TH_5007620481, symbol jlc_parts:5007620481
- added D1, D2: 1N4148WS, hellen-one-common:SOD-323, symbol hellen-one-common:1N4148WS
- added D10, D7, D8, D9: B5819W, hellen-one-common:SOD-123, symbol hellen-one-common:1N4148WS
- added D3, D4, D5, D6: LED-GREEN-0805, hellen-one-common:LED-0805, symbol hellen-one-common:LED
- added F1: Fuse-Pad-Pad, hellen-one-common:PAD-1206-PAD, symbol hellen-one-common:Fuse-Pad-Pad
- added J1: USB_B_Mini, hellen-one-common:USB-MINI-B-VERTICAL, symbol hellen-one-common:USB_B_Mini
- added M2: Module-power_12and5V-0.1, power-12-5v-0.1:power_12and5V, symbol power_12and5V-0.1:Module-power_12and5V-0.1
- added M3: Module-knock-0.2, knock-0.2:knock, symbol hellen-one-knock-0.2:Module-knock-0.2
- added M4: Module-wbo-0.5, wbo-0.5:wbo, symbol hellen-one-wbo-0.5:Module-wbo-0.5
- added M5: Module-mega-mcu144-0.7, mega-144-07:mega-mcu144, symbol mega-mcu144:Module-mega-mcu144-0.7
- added M6: Module-can-0.1, can-01:can, symbol can:Module-can-0.1
- added M7: Module-vr-max9924-0.1, vr-max9924-0.1:vr-max9924, symbol vr-max9924:Module-vr-max9924-0.1
- added M8: Module-vr-discrete-0.4, vr-discrete-0.4:vr-discrete, symbol vr-discrete-0.4:Module-vr-discrete-0.4
- added R1, R2: 5.1k, hellen-one-common:R0603, symbol hellen-one-common:Res
- added R3: 1.6k, hellen-one-common:R0603, symbol hellen-one-common:Res
- added R4: 750, hellen-one-common:R0603, symbol hellen-one-common:Res
- added R5: 0, hellen-one-common:R0603, symbol hellen-one-common:Res
- added U3: molex_48pin_MRE, conector-mre48:Molex_48_MRE, symbol rusefi_Molex_MRE_Connector:molex_48pin_MRE
Connections:
- new net: D5.2 (K), R3.1
- new net: D2.2 (A), D4.2 (K), R2.1
- new net: M5.E1 (SPI2_SCK/CAN2_TX), M6.V5 (CAN_TX)
- new net: M5.E4 (SPI2_CS/CAN2_RX), M6.V6 (CAN_RX)
- new net: M4.J2 (SEL2), M4.J_VCC2 (PULL_UP2)
- new net: D1.2 (A), D3.2 (K), R1.1
- new net: J1.5 (GND), J1.6 (Shield), R5.1
- new net: D6.2 (K), R4.1
- new net +12V: D1.1 (K), D10.1 (K), D2.1 (K), D3.1 (A), D4.1 (A), D7.1 (K), D8.1 (K), D9.1 (K), F1.1, M2.E2 (V12), U3.12, U3.16
- new net +12V_RAW: F1.2, M2.V1 (V12_PERM), M2.V2 (IN_VIGN), M2.V3 (V12_RAW)
- new net +3V3: D6.1 (A), M5.N32 (V33), M6.V2 (CAN_VIO)
- new net +5V: D5.1 (A), M2.E4 (V5), M2.E5 (EN_5VP), M4.W1 (V5_IN), M5.N31 (VCC), M7.E4 (V5_IN)
- new net +5VA: M3.E1 (V5A), M5.N30 (V5A_SWITCHABLE), M6.V1 (V5)
- new net +5VP: M2.V4 (5VP), U3.30, U3.31
- new net +ETB: M5.E17 (OUT_PWM2)
- new net -ETB: M5.E16 (OUT_PWM3)
- new net CAN+: M4.W4 (CANH), M5.W12 (CANH)
- new net CAN-: M4.W3 (CANL), M5.W13 (CANL)
- new net CAN_H: M6.S2 (CANH), U3.39
- new net CAN_L: M6.S1 (CANL), U3.34
- new net CHECK_ENGINE: M5.E22 (OUT_IO8)
- new net EGT+: U3.47
- new net EGT-: U3.43
- new net ETB_EN: M5.E13 (OUT_IO12)
- new net FUEL_CONSUM: M5.E25 (OUT_PWM7)
- new net FUEL_PUMP_RELAY: M5.E8 (OUT_IO1)
- new net GND: M2.S1 (GND), M3.E2 (GND), M4.E6 (LSU_H-), M4.G (GND), M5.G (GND), M6.E1 (GND), M7.G (GND), R1.2, R2.2, R3.2, R4.2, R5.2, U3.4, U3.8
- new net GNDA: M5.W1 (GNDA), U3.37, U3.38, U3.41, U3.42, U3.45, U3.46
- new net IDLE: M5.E21 (OUT_IO4)
- new net IGN1: M5.W11 (IGN1)
- new net IGN2: M5.W10 (IGN2)
- new net IGN3: M5.W9 (IGN3)
- new net IGN4: M5.W8 (IGN4)
- new net IGN5: M5.W7 (IGN5)
- new net IGN6: M5.W6 (IGN6)
- new net INJ1: M5.E19 (OUT_INJ1)
- new net INJ2: M5.E18 (OUT_INJ2)
- new net INJ3: M5.E29 (OUT_INJ3)
- new net INJ4: M5.E30 (OUT_INJ4)
- new net INJ5: M5.E31 (OUT_INJ5)
- new net INJ6: M5.E32 (OUT_INJ6)
- new net IN_A1: M5.S15 (IN_O2S2)
- new net IN_A2: M5.S19 (IN_MAP3)
- new net IN_A3: M5.S11 (IN_AUX3)
- new net IN_A4: M5.S18 (IN_RES3)
- new net IN_AFR: M5.S16 (IN_O2S)
- new net IN_CAM1: M5.S24 (IN_CAM), U3.20
- new net IN_CAM2: M5.S10 (IN_AUX4)
- new net IN_CLT: M5.S28 (IN_CLT), U3.24
- new net IN_CRANK: M5.S22 (IN_CRANK), M7.E3 (OUT)
- new net IN_CRANK+: M7.W2 (VR+), U3.26
- new net IN_CRANK-: M7.W1 (VR-), U3.29
- new net IN_D1: M5.S4 (IN_D1)
- new net IN_D2: M5.S3 (IN_D2)
- new net IN_D3: M5.S2 (IN_D3)
- new net IN_D4: M5.S1 (IN_D4)
- new net IN_IAT: M5.S26 (IN_IAT), U3.23
- new net IN_KNOCK1: M3.E3 (OUT_KNOCK), M5.S23 (IN_KNOCK)
- new net IN_KNOCK1_RAW: M3.W1 (IN_KNOCK), U3.33
- new net IN_MAF: M5.S21 (IN_MAP1)
- new net IN_MAP2: M5.S20 (IN_MAP2), U3.19
- new net IN_PPS1: M5.S31 (IN_PPS), U3.28
- new net IN_PPS2: M5.S12 (IN_AUX2)
- new net IN_RES1: M5.S17 (IN_RES1)
- new net IN_RES2: M5.S14 (IN_RES2)
- new net IN_TPS1: M5.S30 (IN_TPS), U3.27
- new net IN_TPS2: M5.S13 (IN_AUX1)
- new net IN_VSS: M5.S25 (IN_VSS)
- new net LSU_CALIBR_RES: M4.E4 (LSU_Rtrim), U3.21
- new net LSU_HEAT-: M4.E5 (LSU_H+), U3.22
- new net LSU_PUMP_I: M4.E3 (LSU_Ip), U3.18
- new net LSU_SENSOR_U: M4.E1 (LSU_Un), U3.17
- new net LSU_SENSOR_U/PUMP_I: M4.E2 (LSU_Vm), U3.25
- new net MAIN_RELAY: M5.E6 (OUT_IO3)
- new net OUT1: M5.E7 (OUT_IO5)
- new net OUT2: M5.E9 (OUT_IO6)
- new net OUT3: M5.E28 (OUT_PWM8)
- new net OUT_BUZER: D10.2 (A), U3.36
- new net OUT_FUEL_PUMP_RELAY: D7.2 (A), U3.48
- new net OUT_IGN1: U3.1
- new net OUT_IGN2: U3.5
- new net OUT_IGN3: U3.2
- new net OUT_IGN4: U3.6
- new net OUT_IGN5: U3.3
- new net OUT_IGN6: U3.7
- new net OUT_INJ1: U3.9
- new net OUT_INJ2: U3.13
- new net OUT_INJ3: U3.10
- new net OUT_INJ4: U3.14
- new net OUT_INJ5: U3.11
- new net OUT_INJ6: U3.15
- new net OUT_TACH: D9.2 (A), U3.32
- new net OUT_WASTEGATE: D8.2 (A), U3.44
- new net RX1: M5.N24 (UART8_RX)
- new net RX2: M5.N18 (UART2_RX)
- new net SPI3_CS: M5.N10 (SPI3_CS)
- new net SPI3_MISO: M5.N12 (SPI3_MISO)
- new net SPI3_MOSI: M5.N13 (SPI3_MOSI)
- new net SPI3_SCK: M5.N11 (SPI3_SCK)
- new net TACH: M5.E27 (OUT_PWM1)
- new net THRESHOLD_VR: M5.E26 (OUT_PWM6), M7.E1 (NC)
- new net TX1: M5.N25 (UART8_TX)
- new net TX2: M5.N17 (UART2_TX)
- new net USBM: J1.2 (D-), M5.N2 (USBM), U3.35
- new net USBP: J1.3 (D+), M5.N3 (USBP), U3.40
- new net VBAT: M5.N27 (VBAT)
- new net VBUS: J1.1 (VBUS), M5.N4 (VBUS)
- new net VIGN: M2.E3 (VIGN), M5.N26 (IN_VIGN)
- new net VREF2: M3.W2 (VREF), M5.S5 (VREF2)
- new net VR_ANALOG: M5.S9 (IN_SENS1), M7.E2 (NC)
- new net VVT1_1: M5.E10 (OUT_IO10)
- new net VVT1_2: M5.E23 (OUT_IO7)
- new net VVT2_B1: M5.E14 (OUT_PWM5)
- new net VVT2_B2: M5.E15 (OUT_PWM4)
- new net WASTEGATE: M5.E12 (OUT_IO2)
- no-connect marks 0 -> 45
Other:
- added sheet EGT (egt.kicad_sch)
- added sheet Ignition (IGN6.kicad_sch)
- added sheet Injector (INJ6.kicad_sch)
- added sheet LOW_SIDE (LOW_SIDE.kicad_sch)
- note added: "#1"
- note added: "Flyback diodes"
- note added: "LEDs"
- note added: "Power"

Commit message: wew
Parts:
- removed D1, D2: 1N4148WS, hellen-one-common:SOD-323, symbol hellen-one-common:1N4148WS
- removed D10, D7, D8, D9: B5819W, hellen-one-common:SOD-123, symbol hellen-one-common:1N4148WS
- removed D3, D4, D5, D6: LED-GREEN-0805, hellen-one-common:LED-0805, symbol hellen-one-common:LED
- removed F1: Fuse-Pad-Pad, hellen-one-common:PAD-1206-PAD, symbol hellen-one-common:Fuse-Pad-Pad
- removed J1: USB_B_Mini, hellen-one-common:USB-MINI-B-VERTICAL, symbol hellen-one-common:USB_B_Mini
- removed M2: Module-power_12and5V-0.1, power-12-5v-0.1:power_12and5V, symbol power_12and5V-0.1:Module-power_12and5V-0.1
- removed M3: Module-knock-0.2, knock-0.2:knock, symbol hellen-one-knock-0.2:Module-knock-0.2
- removed M4: Module-wbo-0.5, wbo-0.5:wbo, symbol hellen-one-wbo-0.5:Module-wbo-0.5
- removed M5: Module-mega-mcu144-0.7, mega-144-07:mega-mcu144, symbol mega-mcu144:Module-mega-mcu144-0.7
- removed M6: Module-can-0.1, can-01:can, symbol can:Module-can-0.1
- removed M7: Module-vr-max9924-0.1, vr-max9924-0.1:vr-max9924, symbol vr-max9924:Module-vr-max9924-0.1
- removed M8: Module-vr-discrete-0.4, vr-discrete-0.4:vr-discrete, symbol vr-discrete-0.4:Module-vr-discrete-0.4
- removed R1, R2: 5.1k, hellen-one-common:R0603, symbol hellen-one-common:Res
- removed R3: 1.6k, hellen-one-common:R0603, symbol hellen-one-common:Res
- removed R4: 750, hellen-one-common:R0603, symbol hellen-one-common:Res
- removed R5: 0, hellen-one-common:R0603, symbol hellen-one-common:Res
- removed U3: molex_48pin_MRE, conector-mre48:Molex_48_MRE, symbol rusefi_Molex_MRE_Connector:molex_48pin_MRE
- added M1: Module-vr-max9924-0.1, hellen-one-vr-max9924-0.1:vr-max9924, symbol vr-max9924:Module-vr-max9924-0.1
Connections:
- no-connect marks 45 -> 0
Other:
- removed sheet EGT
- removed sheet Ignition
- removed sheet Injector
- removed sheet LOW_SIDE
- note removed: "#1"
- note removed: "Flyback diodes"
- note removed: "LEDs"
- note removed: "Power"
